File: Voyager60.kicad_pcb (KiCad board)
At the start: 2 copper layers, 231 parts, among them Q1 2N7002, SW1 6x6x5mm, U1 ATmega32U4, U2 PRTR5V0U2X, Y1 16Mhz

Commit message: Progress
Parts:
- added REF**: 60_Outline, locallib:60_Outline-Modded, F.Cu at (165.1, 69.8)
- USB1: footprint Type-C:HRO-TYPE-C-31-M-12 -> Type-C:HRO-TYPE-C-31-M-12-Assembly
- moved D31 443.1 mm to (26.2, 69.8), turned to 90 degrees
- moved D1 426.2 mm to (24.6, 31.8), turned to 90 degrees
- moved D2 388.1 mm to (57.9, 31.8), turned to 90 degrees
- moved D16 387.7 mm to (28.6, 50.8), turned to 90 degrees
- moved D4 377.9 mm to (96.0, 31.8), turned to 90 degrees
- moved D17 372.6 mm to (67.5, 50.8), turned to 90 degrees
- moved D32 371.0 mm to (72.2, 69.8), turned to 90 degrees
- moved D3 364.4 mm to (77.0, 31.8), turned to 90 degrees
- moved D5 359.5 mm to (115.1, 31.8), turned to 90 degrees
- moved D18 348.9 mm to (86.5, 50.8), turned to 90 degrees
- moved D19 325.1 mm to (105.6, 50.8), turned to 90 degrees
- moved D7 322.6 mm to (153.2, 31.8), turned to 90 degrees
- moved D33 319.9 mm to (91.3, 69.8), turned to 90 degrees
- moved D6 312.5 mm to (134.1, 31.8), turned to 90 degrees
- moved D8 306.2 mm to (172.2, 31.8), turned to 90 degrees
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Other:
- board outline added: 285 x 95.1 mm

Commit message: Place components
Parts:
- added D44: SOD-123, Diodes_SMD:D_SOD-123, B.Cu at (66.7, 88.9)
- added D58: SOD-123, Diodes_SMD:D_SOD-123, B.Cu at (122.2, 108.0)
- added D62: SOD-123, Diodes_SMD:D_SOD-123, B.Cu at (193.7, 108.0)
- added K_SHIFT2: MX-1.25U, MX_Alps_Hybrid:MXOnly-1.25U, F.Cu at (34.1, 88.9)
- added K_SHIFT3: MX-1U, MX_Alps_Hybrid:MXOnly-1U, F.Cu at (55.6, 88.9)
- added K_SPACE3: MX-2.25U, MX_Alps_Hybrid:MXOnly-2.25U-ReversedStabilizers, F.Cu at (115.1, 108.0)
- added K_SPACE4: MX-2.75U, MX_Alps_Hybrid:MXOnly-2.75U-ReversedStabilizers, F.Cu at (186.5, 108.0)
- added K_SPACE5: MX-1.25U, MX_Alps_Hybrid:MXOnly-1.25U-FLIPPED, F.Cu at (148.4, 108.0)
- added R44: 1k, Resistors_SMD:R_0805, B.Cu at (62.7, 94.5)
- added R58: 1k, Resistors_SMD:R_0805, B.Cu at (122.2, 113.5)
- added R62: 1k, Resistors_SMD:R_0805, B.Cu at (193.7, 113.5)
- C2, C3, C4, C5, C6, C7, C8: footprint Capacitors_SMD:C_0805 -> Capacitors_SMD:C_0603
- K_ALT2, K_RALT3: footprint MX_Alps_Hybrid:MXOnly-1.5U -> MX_Alps_Hybrid:MXOnly-1.5U-FLIPPED
- K_RALT2, K_RMENU2: footprint MX_Alps_Hybrid:MXOnly-1.25U -> MX_Alps_Hybrid:MXOnly-1.25U-FLIPPED
- K_RCTRL1, K_WIN2: footprint MX_Alps_Hybrid:MXOnly-1U -> MX_Alps_Hybrid:MXOnly-1U-FLIPPED
- K_RSHIFT1: footprint MX_Alps_Hybrid:MXOnly-2.75U -> MX_Alps_Hybrid:MXOnly-2.75U-FLIPPED
- SW1: value 6x6x5mm -> 5.2x5.2mm; footprint Molex-0548190589:PushButton_6x6mm_TH_Pretty -> Molex-0548190589:SKQG-1155865
- U1: value ATmega32U4 -> ATmega32U4-MU; footprint Housings_QFP:TQFP-44_10x10mm_Pitch0.8mm -> Housings_DFN_QFN:QFN-44-1EP_7x7mm_Pitch0.5mm
- moved R73 547.9 mm to (32.4, 40.5)
- moved R74 537.6 mm to (47.6, 31.8)
- moved F1 529.5 mm to (35.9, 40.0)
- moved R31 522.8 mm to (26.2, 71.4)
- moved C8 512.5 mm to (47.5, 56.8)
- moved R71 511.2 mm to (58.7, 73.0)
- moved R18 500.5 mm to (86.5, 56.4)
- moved R70 499.5 mm to (81.0, 41.3), turned to 0 degrees
- moved R1 498.2 mm to (24.6, 26.2)
- moved U2 495.7 mm to (40.9, 32.6), turned to 270 degrees
- moved U1 493.8 mm to (51.5, 66.1), turned to 0 degrees
- moved R16 486.4 mm to (28.6, 56.4)
- moved R45 483.8 mm to (66.7, 94.5)
- moved R19 483.5 mm to (105.6, 56.4)
- moved SW1 481.8 mm to (88.9, 42.9), turned to 0 degrees
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Connections:
- K_,1 pad 1: COL8 -> COL9
- K_.1 pad 1: COL9 -> COL10
- K_/1 pad 1: COL10 -> COL11
- K_B1 pad 1: COL5 -> COL6
- K_C1 pad 1: COL3 -> COL4
- K_M1 pad 1: COL7 -> COL8
- K_N1 pad 1: COL6 -> COL7
- K_RSHIFT1 pad 1: COL11 -> COL12
- K_V1 pad 1: COL4 -> COL5
- K_X1 pad 1: COL2 -> COL3
- K_Z1 pad 1: COL1 -> COL2
- R70 pad 1: +5V -> Net-(R70-Pad1)
- U2 pad 2: Net-(R67-Pad2) -> Net-(R68-Pad2)
- U2 pad 3: Net-(R68-Pad2) -> Net-(R67-Pad2)
Routing:
- net Net-(R68-Pad2): track 0.00 -> 12.2 mm
- net Net-(R67-Pad2): track 0.00 -> 10.9 mm

Commit message: Continue routing
Parts:
- removed D15: SOD-123, Diodes_SMD:D_SOD-123
- removed K_EX1, K_RALT1, K_RMENU1, K_RWIN1, K_SRSHIFT4: MX-1U, MX_Alps_Hybrid:MXOnly-1U
- removed K_RCTRL1: MX-1U, MX_Alps_Hybrid:MXOnly-1U-FLIPPED
- removed K_SRSHIFT3: MX-1.75U, MX_Alps_Hybrid:MXOnly-1.75U
- removed R15: 1k, Resistors_SMD:R_0805
- K_#1, K_#10, K_#2, K_#3, K_#4, K_#5, K_#6, K_#7, K_#8, K_#9, K_'1, K_,1, K_-1, K_.1, K_/1, K_;1, K_=1, K_A1, K_B1, K_C1, K_D1, K_E1, K_ESC1, K_F1, K_G1, K_H1, K_I1, K_J1, K_K1, K_L1, K_M1, K_N1, K_O1, K_P1, K_Q1, K_R1, K_RWIN3, K_S1, K_SBACK1, K_SBACK2, K_SHIFT3, K_SRSHIFT2, K_T1, K_U1, K_V1, K_W1, K_X1, K_Y1, K_Z1, K_[1, K_\2, K_]1: footprint MX_Alps_Hybrid:MXOnly-1U -> MX_Alps_Hybrid:MX-1U
- K_ALT1, K_CTRL1, K_RCTRL2, K_RWIN2, K_SHIFT2, K_WIN1: footprint MX_Alps_Hybrid:MXOnly-1.25U -> MX_Alps_Hybrid:MX-1.25U
- K_ALT2, K_CTRL2, K_RALT3: footprint MX_Alps_Hybrid:MXOnly-1.5U-FLIPPED -> MX_Alps_Hybrid:MX-1.5U-FLIPPED
- K_BACK1: footprint MX_Alps_Hybrid:MXOnly-2U -> MX_Alps_Hybrid:MX-2U
- K_CAPS1, K_SRSHIFT1: footprint MX_Alps_Hybrid:MXOnly-1.75U -> MX_Alps_Hybrid:MX-1.75U
- K_CAPS2, K_RALT2, K_RMENU2, K_SPACE5: footprint MX_Alps_Hybrid:MXOnly-1.25U-FLIPPED -> MX_Alps_Hybrid:MX-1.25U-FLIPPED
- K_ENTER1, K_SHIFT1: footprint MX_Alps_Hybrid:MXOnly-2.25U -> MX_Alps_Hybrid:MX-2.25U
- K_ENTER2: footprint MX_Alps_Hybrid:MXOnly-ISO-ROTATED-ReversedStabilizers -> MX_Alps_Hybrid:MX-ISO-ReversedStabilizers
- K_RCTRL3: footprint MX_Alps_Hybrid:MXOnly-1.5U -> MX_Alps_Hybrid:MX-1.5U-FLIPPED
- K_RSHIFT1: footprint MX_Alps_Hybrid:MXOnly-2.75U-FLIPPED -> MX_Alps_Hybrid:MX-2.75U-FLIPPED
- K_SPACE1: footprint MX_Alps_Hybrid:MXOnly-7U-ReversedStabilizers -> MX_Alps_Hybrid:MX-7U-ReversedStabilizers
- K_SPACE2: footprint MX_Alps_Hybrid:MXOnly-6.25U-ReversedStabilizers -> MX_Alps_Hybrid:MX-6.25U-ReversedStabilizers
- K_SPACE3: footprint MX_Alps_Hybrid:MXOnly-2.25U-ReversedStabilizers -> MX_Alps_Hybrid:MX-2.25U-ReversedStabilizers
- K_SPACE4: footprint MX_Alps_Hybrid:MXOnly-2.75U-ReversedStabilizers -> MX_Alps_Hybrid:MX-2.75U-ReversedStabilizers
- K_TAB1, K_\1: footprint MX_Alps_Hybrid:MXOnly-1.5U -> MX_Alps_Hybrid:MX-1.5U
- K_WIN2: footprint MX_Alps_Hybrid:MXOnly-1U-FLIPPED -> MX_Alps_Hybrid:MX-1U-FLIPPED
- moved D45 36.5 mm to (26.2, 88.9)
- moved R44 36.5 mm to (26.2, 94.5)
- moved C4 12.1 mm to (46.7, 60.7), turned to 0 degrees
- moved D44 3.97 mm to (62.7, 88.9)
- moved R45 3.97 mm to (62.7, 94.5)
- moved C3 1.20 mm to (57.3, 61.1)
- moved R71 1.02 mm to (58.8, 72.0), turned to 180 degrees
- moved C6 0.77 mm to (45.2, 65.4)
- moved F1 0.48 mm to (35.9, 40.5)
- turned C8 to 270 degrees
Connections:
- net COL14 renamed Net-(U1-Pad41)
- K_ENTER2 pad 1: Net-(K_ENTER2-Pad1) -> COL13
- K_ENTER2 pad 2: Net-(K_ENTER2-Pad2) -> Net-(D43-Pad2)
- K_ENTER2 pad 3: Net-(K_ENTER2-Pad3) -> +5V
- K_ENTER2 pad 4: Net-(K_ENTER2-Pad4) -> Net-(K_ENTER1-Pad4)
- K_RALT2 pad 1: Net-(K_RALT2-Pad1) -> COL10
- K_RALT2 pad 2: Net-(K_RALT2-Pad2) -> Net-(D63-Pad2)
- K_RALT2 pad 3: Net-(K_RALT2-Pad3) -> +5V
- K_RALT3 pad 1: Net-(K_RALT3-Pad1) -> COL11
- K_RALT3 pad 2: Net-(K_RALT3-Pad2) -> Net-(D64-Pad2)
- K_RALT3 pad 3: Net-(K_RALT3-Pad3) -> +5V
- K_RCTRL2 pad 1: Net-(K_RCTRL2-Pad1) -> COL13
- K_RCTRL2 pad 2: Net-(K_RCTRL2-Pad2) -> Net-(D65-Pad2)
- K_RCTRL2 pad 3: Net-(K_RCTRL2-Pad3) -> +5V
- K_RCTRL3 pad 1: Net-(K_RCTRL3-Pad1) -> COL13
- K_RCTRL3 pad 2: Net-(K_RCTRL3-Pad2) -> Net-(D65-Pad2)
- K_RCTRL3 pad 3: Net-(K_RCTRL3-Pad3) -> +5V
- K_RCTRL3 pad 4: Net-(K_RCTRL3-Pad4) -> Net-(K_RCTRL2-Pad4)
- K_RMENU2 pad 1: Net-(K_RMENU2-Pad1) -> COL12
- K_RMENU2 pad 2: Net-(K_RMENU2-Pad2) -> Net-(D30-Pad2)
- K_RMENU2 pad 3: Net-(K_RMENU2-Pad3) -> +5V
- K_RWIN2 pad 1: Net-(K_RWIN2-Pad1) -> COL11
- K_RWIN2 pad 2: Net-(K_RWIN2-Pad2) -> Net-(D64-Pad2)
- K_RWIN2 pad 3: Net-(K_RWIN2-Pad3) -> +5V
- K_RWIN2 pad 4: Net-(K_RWIN2-Pad4) -> Net-(K_RALT3-Pad4)
- K_RWIN3 pad 1: Net-(K_RWIN3-Pad1) -> COL12
- K_RWIN3 pad 2: Net-(K_RWIN3-Pad2) -> Net-(D30-Pad2)
- K_RWIN3 pad 3: Net-(K_RWIN3-Pad3) -> +5V
- K_RWIN3 pad 4: Net-(K_RWIN3-Pad4) -> Net-(K_RMENU2-Pad4)
- K_SPACE1 pad 1: COL5 -> COL6
- K_SPACE2 pad 1: Net-(D61-Pad2) -> COL6
- K_SPACE2 pad 2: COL5 -> Net-(D61-Pad2)
- K_SPACE3 pad 1: COL3 -> COL4
- K_SPACE4 pad 1: COL7 -> COL8
- K_SPACE5 pad 1: Net-(K_SPACE5-Pad1) -> Net-(D61-Pad2)
- K_SPACE5 pad 2: Net-(K_SPACE5-Pad2) -> COL6
- K_SPACE5 pad 3: Net-(K_SPACE5-Pad3) -> +5V
- K_SPACE5 pad 4: Net-(K_SPACE5-Pad4) -> Net-(K_SPACE1-Pad4)
- K_SRSHIFT1 pad 1: Net-(K_SRSHIFT1-Pad1) -> COL12
- K_SRSHIFT1 pad 2: Net-(K_SRSHIFT1-Pad2) -> Net-(D56-Pad2)
- K_SRSHIFT1 pad 3: Net-(K_SRSHIFT1-Pad3) -> +5V
- K_SRSHIFT1 pad 4: Net-(K_SRSHIFT1-Pad4) -> Net-(K_RSHIFT1-Pad4)
- K_\2 pad 1: Net-(K_\2-Pad1) -> COL13
- K_\2 pad 2: Net-(K_\2-Pad2) -> Net-(D29-Pad2)
- K_\2 pad 3: Net-(K_\2-Pad3) -> +5V
- K_\2 pad 4: Net-(K_\2-Pad4) -> Net-(K_\1-Pad4)
- R30 pad 1: Net-(K_RMENU1-Pad4) -> Net-(K_RMENU2-Pad4)
- R63 pad 1: Net-(K_RALT1-Pad4) -> Net-(K_RALT2-Pad4)
- R64 pad 1: Net-(K_RWIN1-Pad4) -> Net-(K_RALT3-Pad4)
- R65 pad 1: Net-(K_RCTRL1-Pad4) -> Net-(K_RCTRL2-Pad4)
- R70 pad 1: Net-(R70-Pad1) -> +5V
- U1 pad 10: Net-(U1-Pad10) -> ROW1
- U1 pad 11: ROW0 -> ROW2
- U1 pad 18: ROW1 -> Net-(U1-Pad18)
- U1 pad 19: ROW2 -> ROW3
- U1 pad 20: ROW3 -> ROW4
- U1 pad 21: ROW4 -> COL13
- U1 pad 22: COL0 -> COL12
- U1 pad 25: COL1 -> COL11
- U1 pad 26: COL2 -> COL10
- U1 pad 27: COL3 -> COL9
- U1 pad 28: COL4 -> COL8
- U1 pad 29: COL5 -> COL7
- U1 pad 31: COL7 -> COL5
- U1 pad 32: COL8 -> COL4
- U1 pad 36: COL9 -> COL1
- U1 pad 37: COL10 -> COL2
- U1 pad 38: COL11 -> COL0
- U1 pad 39: COL12 -> COL3
- U1 pad 40: COL13 -> Net-(U1-Pad40)
- U1 pad 9: Net-(U1-Pad9) -> ROW0
Routing:
- net COL8: track 0.00 -> 365.7 mm
- net COL7: track 0.00 -> 363.2 mm
- net COL6: track 0.00 -> 357.0 mm
- net COL13: track 0.00 -> 353.8 mm
- net COL10: track 0.00 -> 329.0 mm, vias 0 -> 1
- net COL9: track 0.00 -> 328.1 mm
- net COL11: track 0.00 -> 311.4 mm, vias 0 -> 1
- net COL12: track 0.00 -> 310.9 mm, vias 0 -> 1
- net COL5: track 0.00 -> 279.6 mm
- net ROW3: track 0.00 -> 273.4 mm, vias 0 -> 1
- net ROW4: track 0.00 -> 271.5 mm, vias 0 -> 1
- net ROW2: track 0.00 -> 245.3 mm
- net COL4: track 0.00 -> 243.6 mm
- net ROW1: track 0.00 -> 222.0 mm
- net ROW0: track 0.00 -> 222.0 mm
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
Commit message: Continue routing
Parts:
- moved D64 51.6 mm to (255.6, 108.0)
- moved R44 36.5 mm to (62.7, 94.5)
- moved R45 36.5 mm to (26.2, 94.5)
- moved D30 7.14 mm to (279.4, 108.0)
- moved D55 7.14 mm to (253.2, 88.9)
- moved R30 7.14 mm to (279.4, 113.5)
- moved R55 7.14 mm to (253.2, 94.5)
- moved D65 2.38 mm to (303.2, 108.0)
- moved R65 2.38 mm to (303.2, 113.5)
- moved D63 1.59 mm to (231.8, 108.0)
- moved R63 1.59 mm to (231.8, 113.5)
- moved R64 0.79 mm to (255.6, 113.5)
Connections:
- K_SHIFT2 pad 1: Net-(K_SHIFT2-Pad1) -> COL0
- K_SHIFT2 pad 2: Net-(K_SHIFT2-Pad2) -> Net-(D45-Pad2)
- K_SHIFT2 pad 3: Net-(K_SHIFT2-Pad3) -> +5V
- K_SHIFT2 pad 4: Net-(K_SHIFT2-Pad4) -> Net-(K_SHIFT1-Pad4)
- K_WIN2 pad 1: Net-(D60-Pad2) -> COL1
- K_WIN2 pad 2: COL1 -> Net-(D60-Pad2)
Routing:
- net LEDGND: track 0.00 -> 1156.9 mm
- net +5V: track 16.9 -> 115.2 mm, vias 1 -> 2
- net Net-(D29-Pad2): track 0.00 -> 40.6 mm, vias 0 -> 1
- net Net-(K_\1-Pad4): track 0.00 -> 38.8 mm, vias 0 -> 1
- net Net-(K_SBACK2-Pad4): track 0.00 -> 30.5 mm
- net Net-(D61-Pad2): track 0.00 -> 30.1 mm
- net Net-(K_SPACE1-Pad4): track 0.00 -> 29.0 mm
- net Net-(K_BACK1-Pad4): track 0.00 -> 26.6 mm
- net Net-(D45-Pad2): track 0.00 -> 26.0 mm
- net ROW2: track 245.3 -> 270.3 mm, vias 0 -> 2
- net Net-(K_ENTER1-Pad4): track 0.00 -> 22.0 mm
- net Net-(K_SHIFT1-Pad4): track 0.00 -> 21.8 mm
- net Net-(D31-Pad2): track 0.00 -> 17.5 mm, vias 0 -> 1
- net Net-(D36-Pad2): track 0.00 -> 16.5 mm
- net Net-(K_CAPS1-Pad4): track 0.00 -> 16.3 mm
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- added copper zone on B.Cu, net GND

Commit message: Progress
Parts:
- moved SW1 59.8 mm to (71.4, 100.0)
- moved R70 46.6 mm to (46.8, 73.0), turned to 180 degrees
- moved R71 1.14 mm to (59.9, 72.0)
- moved C4 0.18 mm to (46.6, 60.8), turned to 270 degrees
Connections:
- U1 pad 19: ROW3 -> Net-(U1-Pad19)
- U1 pad 20: ROW4 -> Net-(U1-Pad20)
- U1 pad 37: COL2 -> COL3
- U1 pad 38: COL0 -> COL2
- U1 pad 39: COL3 -> COL0
- U1 pad 40: Net-(U1-Pad40) -> ROW4
- U1 pad 41: Net-(U1-Pad41) -> ROW3
Routing:
- net +5V: track 115.2 -> 1354.6 mm, vias 2 -> 13
- net ROW2: track 270.3 -> 359.3 mm, vias 2 -> 7
- net ROW0: track 222.0 -> 287.2 mm, vias 0 -> 2
- net GND: track 87.7 -> 135.7 mm, vias 0 -> 2
- net COL12: track 310.9 -> 356.3 mm
- net ROW1: track 222.0 -> 266.6 mm
- net ROW4: track 269.1 -> 309.9 mm, vias 1 -> 2
- net COL3: track 115.5 -> 146.1 mm
- net ROW3: track 274.1 -> 296.0 mm, vias 1 -> 2
- net Net-(R70-Pad2): track 6.10 -> 16.3 mm, vias 0 -> 2
- net Net-(R74-Pad2): track 0.00 -> 8.82 mm, vias 0 -> 2
- net VCC: track 13.2 -> 20.9 mm, vias 0 -> 2
- net Net-(R71-Pad2): track 0.00 -> 6.74 mm, vias 0 -> 2
- net COL0: track 115.5 -> 118.7 mm
- net Net-(R69-Pad2): track 48.1 -> 45.1 mm
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
Commit message: Progress
Parts:
- turned R16 to 270 degrees
- turned R43 to 270 degrees
Routing:
- net +5V: track 1354.6 -> 1698.4 mm, vias 13 -> 12
- net LEDGND: track 1157.0 -> 1236.0 mm, vias 0 -> 3
- net COL6: track 354.3 -> 369.3 mm
- net ROW1: track 266.6 -> 280.9 mm, vias 0 -> 2
- net COL13: track 351.4 -> 353.7 mm
- net Net-(K_TAB1-Pad4): track 9.80 -> 10.7 mm
- net ROW0: track 287.2 -> 286.7 mm
- net Net-(K_SRSHIFT2-Pad4): track 12.1 -> 12.6 mm

Commit message: Finish routing
Routing:
- net LEDGND: track 1236.0 -> 1420.0 mm, vias 3 -> 11
- net GND: track 135.7 -> 231.5 mm, vias 2 -> 8
- net Net-(R70-Pad2): track 16.3 -> 68.7 mm, vias 2 -> 4
- net +5V: track 1698.4 -> 1708.1 mm
- net Net-(K_RSHIFT1-Pad4): track 11.0 -> 19.1 mm
- net Net-(D30-Pad2): track 10.6 -> 13.2 mm
- net Net-(D67-Pad2): track 8.21 -> 10.8 mm
- net Net-(D59-Pad2): track 8.21 -> 10.8 mm
- net Net-(D64-Pad2): track 8.28 -> 10.9 mm
- net Net-(D65-Pad2): track 5.82 -> 8.21 mm
- net Net-(D60-Pad2): track 8.21 -> 10.6 mm

Commit message: Route RGBs
Parts:
- added C1: 0.1uF, Capacitors_SMD:C_0603, B.Cu at (54.8, 41.3)
- added C10: 0.1uF, Capacitors_SMD:C_0603, B.Cu at (129.4, 41.3)
- added C11: 0.1uF, Capacitors_SMD:C_0603, B.Cu at (170.7, 41.3)
- added C12: 0.1uF, Capacitors_SMD:C_0603, B.Cu at (211.9, 41.3)
- added C13: 0.1uF, Capacitors_SMD:C_0603, B.Cu at (253.2, 41.3)
- added C14: 0.1uF, Capacitors_SMD:C_0603, B.Cu at (294.5, 41.3)
- added C15: 0.1uF, Capacitors_SMD:C_0603, B.Cu at (281.8, 98.4)
- added C16: 0.1uF, Capacitors_SMD:C_0603, B.Cu at (253.2, 98.4)
- added C17: 0.1uF, Capacitors_SMD:C_0603, B.Cu at (215.1, 98.4)
- added C18: 0.1uF, Capacitors_SMD:C_0603, B.Cu at (162.7, 98.4)
- added C19: 0.1uF, Capacitors_SMD:C_0603, B.Cu at (115.1, 98.4)
- added C20: 0.1uF, Capacitors_SMD:C_0603, B.Cu at (88.1, 98.4)
- added C21: 0.1uF, Capacitors_SMD:C_0603, B.Cu at (49.2, 98.4)
- added C9: 0.1uF, Capacitors_SMD:C_0603, B.Cu at (89.7, 41.3)
- added RGB1: WS2812B, WS2812B:WS2812B, B.Cu at (49.2, 41.3)
- added RGB10: WS2812B, WS2812B:WS2812B, B.Cu at (120.7, 98.4)
- added RGB11: WS2812B, WS2812B:WS2812B, B.Cu at (247.7, 41.3)
- added RGB12: WS2812B, WS2812B:WS2812B, B.Cu at (82.5, 98.4)
- added RGB13: WS2812B, WS2812B:WS2812B, B.Cu at (288.9, 41.3)
- added RGB14: WS2812B, WS2812B:WS2812B, B.Cu at (43.7, 98.4)
- added RGB2: WS2812B, WS2812B:WS2812B, B.Cu at (287.3, 98.4)
- added RGB3: WS2812B, WS2812B:WS2812B, B.Cu at (84.1, 41.3)
- added RGB4: WS2812B, WS2812B:WS2812B, B.Cu at (247.7, 98.4)
- added RGB5: WS2812B, WS2812B:WS2812B, B.Cu at (123.8, 41.3)
- added RGB6: WS2812B, WS2812B:WS2812B, B.Cu at (209.6, 98.4)
- added RGB7: WS2812B, WS2812B:WS2812B, B.Cu at (165.1, 41.3)
- added RGB8: WS2812B, WS2812B:WS2812B, B.Cu at (168.3, 98.4)
- added RGB9: WS2812B, WS2812B:WS2812B, B.Cu at (206.4, 41.3)
- moved R10 2.38 mm to (212.7, 37.3)
- moved D44 1.59 mm to (62.7, 87.3)
- moved D46 1.59 mm to (81.8, 87.3)
- moved D47 1.59 mm to (100.8, 87.3)
- moved D48 1.59 mm to (119.9, 87.3)
- moved D49 1.59 mm to (138.9, 87.3)
- moved D50 1.59 mm to (158.0, 87.3)
- moved D51 1.59 mm to (177.0, 87.3)
- moved D52 1.59 mm to (196.1, 87.3)
- moved D53 1.59 mm to (215.1, 87.3)
- moved D54 1.59 mm to (234.2, 87.3)
- moved D55 1.59 mm to (253.2, 87.3)
- moved D56 1.59 mm to (264.3, 87.3)
- moved D57 1.59 mm to (288.9, 87.3)
- moved D12 1.59 mm to (248.4, 30.2)
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Connections:
- U1 pad 20: Net-(U1-Pad20) -> RGBLED
Routing:
- net GND: track 231.5 -> 865.7 mm, vias 8 -> 24
- net +5V: track 1708.1 -> 1795.4 mm, vias 12 -> 13
- net Net-(RGB13-Pad2): track 0.00 -> 71.5 mm, vias 0 -> 2
- net Net-(RGB10-Pad4): track 0.00 -> 56.0 mm
- net Net-(RGB12-Pad2): track 0.00 -> 53.4 mm
- net Net-(RGB6-Pad2): track 0.00 -> 48.4 mm
- net Net-(RGB10-Pad2): track 0.00 -> 48.2 mm
- net RGBLED: track 0.00 -> 47.7 mm, vias 0 -> 2
- net Net-(RGB4-Pad2): track 0.00 -> 47.4 mm
- net Net-(RGB2-Pad2): track 0.00 -> 47.0 mm
- net Net-(RGB11-Pad4): track 0.00 -> 37.9 mm
- net Net-(RGB5-Pad2): track 0.00 -> 37.9 mm
- net Net-(RGB7-Pad2): track 0.00 -> 37.9 mm
- net Net-(RGB11-Pad2): track 0.00 -> 37.9 mm
- net Net-(RGB3-Pad2): track 0.00 -> 36.4 mm
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