File: Voyager60.kicad_pcb (KiCad board)
At the start: 2 copper layers, 285 x 95.1 mm, 262 parts, among them Q1 2N7002, SW1 5.2x5.2mm, U1 ATmega32U4-MU, U2 PRTR5V0U2X, Y1 16Mhz

Commit message: Finish routing, add decorations
Parts:
- added G***: LOGO, locallib:ai-ring-6mm, B.Cu at (76.2, 61.1)
- added G***: LOGO, locallib:ai-ring-6mm-FancyAss, F.Cu at (263.5, 98.4)
- added G***: LOGO, locallib:ai-ring-6mm-FancyAss-Mask, F.Cu at (263.5, 98.4)
Routing:
- net LEDGND: track 1408.1 -> 1409.4 mm
- net GND: track 865.7 -> 864.6 mm
Other:
- board text added: "60"
- board text added: "PCB Revision 1.0"
- board text added: "VOYAGER"
- board text added: "kb.ai03.me"
