File: Voyager60.kicad_pcb (KiCad board)
At the start: 2 copper layers, 285 x 95.1 mm, 265 parts, among them Q1 2N7002, SW1 5.2x5.2mm, U1 ATmega32U4-MU, U2 PRTR5V0U2X, Y1 16Mhz

Commit message: Make alps variant
Parts:
- removed Q1: 2N7002, TO_SOT_Packages_SMD:SOT-23
- removed R1, R10, R11, R12, R13, R14, R16, R17, R18, R19, R2, R20, R21, R22, R23, R24, R25, R26, R27, R28, R29, R3, R30, R31, R32, R33, R34, R35, R36, R37, R38, R39, R4, R40, R41, R42, R43, R44, R45, R46, R47, R48, R49, R5, R50, R51, R52, R53, R54, R55, R56, R57, R58, R59, R6, R60, R61, R62, R63, R64, R65, R69, R7, R72, R75, R8, R9: 1k, Resistors_SMD:R_0805
- added K_ALT3: MX-1.5U, MX_Alps_Hybrid:ALPS-1.5U, F.Cu at (88.9, 108.0)
- added K_CAPS3: MX-1.5U, MX_Alps_Hybrid:ALPS-1.5U, F.Cu at (36.5, 69.8)
- added K_ENTER3: MX-1U, MX_Alps_Hybrid:ALPS-1U, F.Cu at (298.4, 60.3)
- added K_ENTER4: MX-1U, MX_Alps_Hybrid:ALPS-1U, F.Cu at (293.7, 60.3)
- added K_ESC2: MX-1U, MX_Alps_Hybrid:ALPS-1U, F.Cu at (31.8, 31.8)
- added K_RALT1: MX-1.5U, MX_Alps_Hybrid:ALPS-1.5U, F.Cu at (241.3, 108.0)
- added K_RWIN1: MX-1.25U, MX_Alps_Hybrid:ALPS-1.25U, F.Cu at (267.5, 108.0)
- added K_WIN3: MX-1.25U, MX_Alps_Hybrid:ALPS-1.25U, F.Cu at (62.7, 108.0)
- K_#1, K_#10, K_#2, K_#3, K_#4, K_#5, K_#6, K_#7, K_#8, K_#9, K_'1, K_,1, K_-1, K_.1, K_/1, K_;1, K_=1, K_A1, K_B1, K_C1, K_D1, K_E1, K_ESC1, K_F1, K_G1, K_H1, K_I1, K_J1, K_K1, K_L1, K_M1, K_N1, K_O1, K_P1, K_Q1, K_R1, K_RWIN3, K_S1, K_SBACK1, K_SBACK2, K_SHIFT3, K_SRSHIFT2, K_T1, K_U1, K_V1, K_W1, K_X1, K_Y1, K_Z1, K_[1, K_\2, K_]1: footprint MX_Alps_Hybrid:MX-1U -> MX_Alps_Hybrid:ALPS-1U
- K_ALT1, K_CTRL1, K_RCTRL2, K_RWIN2, K_SHIFT2, K_WIN1: footprint MX_Alps_Hybrid:MX-1.25U -> MX_Alps_Hybrid:ALPS-1.25U
- K_ALT2, K_CTRL2, K_RALT3, K_RCTRL3: footprint MX_Alps_Hybrid:MX-1.5U-FLIPPED -> MX_Alps_Hybrid:ALPS-1.5U
- K_BACK1: footprint MX_Alps_Hybrid:MX-2U -> MX_Alps_Hybrid:ALPS-2U
- K_CAPS1, K_SRSHIFT1: footprint MX_Alps_Hybrid:MX-1.75U -> MX_Alps_Hybrid:ALPS-1.75U
- K_CAPS2, K_RALT2, K_RMENU2, K_SPACE5: footprint MX_Alps_Hybrid:MX-1.25U-FLIPPED -> MX_Alps_Hybrid:ALPS-1.25U
- K_ENTER1, K_SHIFT1: footprint MX_Alps_Hybrid:MX-2.25U -> MX_Alps_Hybrid:ALPS-2.25U
- K_ENTER2: value MX-ISO -> MX-1U; footprint MX_Alps_Hybrid:MX-ISO-ReversedStabilizers -> MX_Alps_Hybrid:ALPS-1U
- K_RSHIFT1: footprint MX_Alps_Hybrid:MX-2.75U-FLIPPED -> MX_Alps_Hybrid:ALPS-2.75U
- K_SPACE1: footprint MX_Alps_Hybrid:MX-7U-ReversedStabilizers -> MX_Alps_Hybrid:ALPS-7U
- K_SPACE2: footprint MX_Alps_Hybrid:MX-6.25U-ReversedStabilizers -> MX_Alps_Hybrid:ALPS-6.25U
- K_SPACE3: footprint MX_Alps_Hybrid:MX-2.25U-ReversedStabilizers -> MX_Alps_Hybrid:ALPS-2.25U
- K_SPACE4: footprint MX_Alps_Hybrid:MX-2.75U-ReversedStabilizers -> MX_Alps_Hybrid:ALPS-2.75U
- K_TAB1, K_\1: footprint MX_Alps_Hybrid:MX-1.5U -> MX_Alps_Hybrid:ALPS-1.5U
- K_WIN2: footprint MX_Alps_Hybrid:MX-1U-FLIPPED -> MX_Alps_Hybrid:ALPS-1U
- moved SW1 58.0 mm to (34.1, 55.6), turned to 90 degrees
- moved D45 40.6 mm to (66.7, 86.5)
- moved D43 27.1 mm to (266.7, 67.5)
- moved D29 24.7 mm to (301.6, 48.4)
- moved D65 19.2 mm to (284.2, 105.6)
- moved C7 18.5 mm to (41.7, 69.8), turned to 270 degrees
- moved C8 16.8 mm to (44.8, 73.4), turned to 0 degrees
- moved Y1 14.5 mm to (44.8, 69.8), turned to 270 degrees
- moved C19 14.3 mm to (129.4, 98.4)
- moved C4 14.0 mm to (48.8, 74.7), turned to 0 degrees
- moved C6 12.7 mm to (52.6, 75.7)
- moved C2 12.6 mm to (57.4, 74.7), turned to 180 degrees
- moved C15 11.1 mm to (292.9, 98.4)
- moved R73 8.90 mm to (34.1, 31.8), turned to 0 degrees
- moved C5 8.85 mm to (57.4, 63.4), turned to 180 degrees
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Connections:
- K_ALT2 pad 1: COL2 -> Net-(D67-Pad2)
- K_ALT2 pad 2: Net-(D67-Pad2) -> COL2
- K_CTRL2 pad 1: COL0 -> Net-(D59-Pad2)
- K_CTRL2 pad 2: Net-(D59-Pad2) -> COL0
- K_RALT3 pad 1: COL11 -> Net-(D64-Pad2)
- K_RALT3 pad 2: Net-(D64-Pad2) -> COL11
- K_RCTRL3 pad 1: COL13 -> Net-(D65-Pad2)
- K_RCTRL3 pad 2: Net-(D65-Pad2) -> COL13
- K_RWIN3 pad 1: COL12 -> Net-(D30-Pad2)
- K_RWIN3 pad 2: Net-(D30-Pad2) -> COL12
Routing:
- net LEDGND: track 1409.4 -> 0.00 mm, vias 11 -> 0
- net +5V: track 1795.4 -> 757.3 mm, vias 13 -> 8
- net ROW1: track 280.9 -> 336.1 mm, vias 2 -> 4
- net Net-(U1-Pad12): track 47.5 -> 0.00 mm, vias 2 -> 0
- net COL2: track 121.4 -> 167.0 mm, vias 1 -> 0
- net COL3: track 146.6 -> 188.2 mm, vias 1 -> 0
- net Net-(K_\1-Pad4): track 39.0 -> 0.00 mm, vias 1 -> 0
- net COL11: track 310.5 -> 348.0 mm, vias 1 -> 0
- net ROW0: track 289.8 -> 325.7 mm, vias 2 -> 4
- net Net-(K_SBACK2-Pad4): track 30.5 -> 0.00 mm
- net Net-(K_SPACE1-Pad4): track 29.0 -> 0.00 mm
- net COL0: track 118.7 -> 145.8 mm
- net Net-(K_BACK1-Pad4): track 26.6 -> 0.00 mm
- net COL6: track 369.3 -> 395.5 mm
- net COL5: track 279.6 -> 303.7 mm
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Other:
- board text added: "60-ALPS"
- board text removed: "60"

Commit message: Push changes
Routing:
- net Net-(D29-Pad2): track 32.6 -> 37.5 mm, vias 0 -> 1
- net ROW1: track 336.1 -> 335.4 mm, vias 4 -> 2
