File: Voyager60.sch (KiCad schematic (older format))
At the start: 261 parts, among them Q1 2N7002, SW1 5.2x5.2mm, U1 ATmega32U4-MU, U2 PRTR5V0U2X, Y1 16Mhz

Commit message: Update bom
Parts:
- U1: symbol MCU_Microchip_ATmega:ATmega32U4-MU -> Voyager60-rescue:ATmega32U4-MU-MCU_Microchip_ATmega
Changed lines of the file:
@@
 	6325 3975 6225 3975
 $Comp
-L MCU_Microchip_ATmega:ATmega32U4-MU U1
+L Voyager60-rescue:ATmega32U4-MU-MCU_Microchip_ATmega U1
 U 1 1 5D93C3AA
 P 8150 7800
